Commit message: cleanup gazebo worlds and add gazebo objects

File: hbrs_environments/hbrs_gazebo_worlds/common/worlds/brsu-c069.urdf.xacro (robot description, xacro)
@@ -5,7 +5,7 @@
 	xmlns:interface="http://playerstage.sourceforge.net/gazebo/xmlschema/#interface"
 	xmlns:xacro="http://playerstage.sourceforge.net/gazebo/xmlschema/#interface"
-	name="brsu_home"
+	name="brsu-c069"
 >
-<xacro:macro name="brsu_home" params="name">
+<xacro:macro name="brsu-c069" params="name">
 <!-- dummy_link -->
 	<link name="dummy_link">
@@ -180,5 +180,5 @@
 			<origin xyz="0 0 0" />
 			<geometry>
-				<!-- <mesh filename="package://hbrs_gazebo_worlds/Media/models/brsu_home/kitchen_counter_1.dae" /> -->
+				<!-- <mesh filename="package://hbrs_gazebo_worlds/common/objects/models/kitchen_counter_1.dae" /> -->
 				<box size="0.62 2.01 0.89" />
 			</geometry>
@@ -208,5 +208,5 @@
 			<origin xyz="0 0 0" />
 			<geometry>
-				<!-- <mesh filename="package://hbrs_gazebo_worlds/Media/models/brsu_home/kitchen_counter_2.dae" /> -->
+				<!-- <mesh filename="package://hbrs_gazebo_worlds/common/objects/models/kitchen_counter_2.dae" /> -->
 				<!-- <box size="0.82 0.53 0.89" /> -->
 				<box size="0.82 0.58 0.89" />
@@ -237,5 +237,5 @@
 			<origin xyz="0 0 0" />
 			<geometry>
-				<!-- <mesh filename="package://hbrs_gazebo_worlds/Media/models/brsu_home/kitchen_counter_3.dae" /> -->
+				<!-- <mesh filename="package://hbrs_gazebo_worlds/common/objects/models/kitchen_counter_3.dae" /> -->
 				<box size="1.915 0.62 0.89" />
 			</geometry>
@@ -265,5 +265,5 @@
 			<origin xyz="0 0 0" />
 			<geometry>
-				<mesh filename="package://hbrs_gazebo_worlds/Media/models/brsu_home/kitchen_fridge.dae" />
+				<mesh filename="package://hbrs_gazebo_worlds/common/objects/models/kitchen_fridge.dae" />
 				<!-- <box size="0.63 0.62 2.325" /> -->
 			</geometry>
@@ -272,5 +272,5 @@
 			<origin xyz="0 0 0" />
 			<geometry>
-				<mesh filename="package://hbrs_gazebo_worlds/Media/models/brsu_home/kitchen_fridge.dae" />
+				<mesh filename="package://hbrs_gazebo_worlds/common/objects/models/kitchen_fridge.dae" />
 				<!-- <box size="0.65 0.64 2.34" /> -->
 			</geometry>
@@ -295,5 +295,5 @@
 			<origin xyz="0 0 0" />
 			<geometry>
-				<mesh filename="package://hbrs_gazebo_worlds/Media/models/brsu_home/lounge_shelf.dae" />
+				<mesh filename="package://hbrs_gazebo_worlds/common/objects/models/lounge_shelf.dae" />
 				<!-- <box size="1.84 0.39 1.84" /> -->
 			</geometry>
@@ -302,5 +302,5 @@
 			<origin xyz="0 0 0" />
 			<geometry>
-				<mesh filename="package://hbrs_gazebo_worlds/Media/models/brsu_home/lounge_shelf.dae" />
+				<mesh filename="package://hbrs_gazebo_worlds/common/objects/models/lounge_shelf.dae" />
 				<!-- <box size="1.86 0.41 1.86" /> -->
 			</geometry>
@@ -324,5 +324,5 @@
 			<origin xyz="0 0 0" />
 			<geometry>
-				<mesh filename="package://hbrs_gazebo_worlds/Media/models/brsu_home/lounge_shelf.dae" />
+				<mesh filename="package://hbrs_gazebo_worlds/common/objects/models/lounge_shelf.dae" />
 				<!-- <box size="1.84 0.39 1.84" /> -->
 			</geometry>
@@ -331,5 +331,5 @@
 			<origin xyz="0 0 0" />
 			<geometry>
-				<mesh filename="package://hbrs_gazebo_worlds/Media/models/brsu_home/lounge_shelf.dae" />
+				<mesh filename="package://hbrs_gazebo_worlds/common/objects/models/lounge_shelf.dae" />
 				<!-- <box size="1.86 0.41 1.86" /> -->
 			</geometry>
@@ -353,5 +353,5 @@
 			<origin xyz="0 0 0" />
 			<geometry>
-				<mesh filename="package://hbrs_gazebo_worlds/Media/models/brsu_home/charger_desk.dae" />
+				<mesh filename="package://hbrs_gazebo_worlds/common/objects/models/charger_desk.dae" />
 				<!-- <box size="0.45 0.45 0.50" /> -->
 			</geometry>
@@ -360,5 +360,5 @@
 			<origin xyz="0 0 0" />
 			<geometry>
-				<mesh filename="package://hbrs_gazebo_worlds/Media/models/brsu_home/charger_desk.dae" />
+				<mesh filename="package://hbrs_gazebo_worlds/common/objects/models/charger_desk.dae" />
 				<!-- <box size="0.47 0.47 0.52" /> -->
 			</geometry>
@@ -382,5 +382,5 @@
 			<origin xyz="0 0 0" />
 			<geometry>
-				<mesh filename="package://hbrs_gazebo_worlds/Media/models/brsu_home/lounge_armchair.dae" />
+				<mesh filename="package://hbrs_gazebo_worlds/common/objects/models/lounge_armchair.dae" />
 				<!-- <cylinder radius="0.45" length="0.64" /> -->
 			</geometry>
@@ -389,5 +389,5 @@
 			<origin xyz="0 0 0" />
 			<geometry>
-				<mesh filename="package://hbrs_gazebo_worlds/Media/models/brsu_home/lounge_armchair.dae" />
+				<mesh filename="package://hbrs_gazebo_worlds/common/objects/models/lounge_armchair.dae" />
 				<!-- <cylinder radius="0.377" length="0.69" /> -->
 			</geometry>
@@ -411,5 +411,5 @@
 			<origin xyz="0 0 0" />
 			<geometry>
-				<mesh filename="package://hbrs_gazebo_worlds/Media/models/brsu_home/lounge_armchair.dae" />
+				<mesh filename="package://hbrs_gazebo_worlds/common/objects/models/lounge_armchair.dae" />
 				<!-- <cylinder radius="0.45" length="0.64" /> -->
 			</geometry>
@@ -418,5 +418,5 @@
 			<origin xyz="0 0 0" />
 			<geometry>
-				<mesh filename="package://hbrs_gazebo_worlds/Media/models/brsu_home/lounge_armchair.dae" />
+				<mesh filename="package://hbrs_gazebo_worlds/common/objects/models/lounge_armchair.dae" />
 				<!-- <cylinder radius="0.377" length="0.69" /> -->
 			</geometry>
@@ -440,5 +440,5 @@
 			<origin xyz="0 0 0" />
 			<geometry>
-				<mesh filename="package://hbrs_gazebo_worlds/Media/models/brsu_home/lounge_armchair_2.dae" />
+				<mesh filename="package://hbrs_gazebo_worlds/common/objects/models/lounge_armchair_2.dae" />
 				<!-- <box size="0.9 0.9 0.65" /> -->
 			</geometry>
@@ -447,5 +447,5 @@
 			<origin xyz="0 0 0" />
 			<geometry>
-				<mesh filename="package://hbrs_gazebo_worlds/Media/models/brsu_home/lounge_armchair_2.dae" />
+				<mesh filename="package://hbrs_gazebo_worlds/common/objects/models/lounge_armchair_2.dae" />
 				<!-- <box size="0.92 0.92 0.67" /> -->
 			</geometry>
@@ -470,5 +470,5 @@
 			<origin xyz="0 0 0" />
 			<geometry>
-				<mesh filename="package://hbrs_gazebo_worlds/Media/models/brsu_home/livingroom_shelf.dae" />
+				<mesh filename="package://hbrs_gazebo_worlds/common/objects/models/livingroom_shelf.dae" />
 				<!-- <box size="2.40 0.43 1.28" /> -->
 			</geometry>
@@ -477,5 +477,5 @@
 			<origin xyz="0 0 0" />
 			<geometry>
-				<mesh filename="package://hbrs_gazebo_worlds/Media/models/brsu_home/livingroom_shelf.dae" />
+				<mesh filename="package://hbrs_gazebo_worlds/common/objects/models/livingroom_shelf.dae" />
 				<!-- <box size="2.42 0.45 1.30" /> -->
 			</geometry>
@@ -499,5 +499,5 @@
 			<origin xyz="0 0 0" />
 			<geometry>
-				<mesh filename="package://hbrs_gazebo_worlds/Media/models/brsu_home/livingroom_couch_1.dae" />
+				<mesh filename="package://hbrs_gazebo_worlds/common/objects/models/livingroom_couch_1.dae" />
 				<!-- <box size="0.98 2.20 0.66" /> -->
 			</geometry>
@@ -506,5 +506,5 @@
 			<origin xyz="0 0 0" />
 			<geometry>
-				<mesh filename="package://hbrs_gazebo_worlds/Media/models/brsu_home/livingroom_couch_1.dae" />
+				<mesh filename="package://hbrs_gazebo_worlds/common/objects/models/livingroom_couch_1.dae" />
 				<!-- <box size="1.00 2.22 0.68" /> -->
 			</geometry>
@@ -528,5 +528,5 @@
 			<origin xyz="0 0 0" />
 			<geometry>
-				<mesh filename="package://hbrs_gazebo_worlds/Media/models/brsu_home/livingroom_couch_2.dae" />
+				<mesh filename="package://hbrs_gazebo_worlds/common/objects/models/livingroom_couch_2.dae" />
 				<!-- <box size="2.81 0.93 0.66" /> -->
 			</geometry>
@@ -535,5 +535,5 @@
 			<origin xyz="0 0 0" />
 			<geometry>
-				<mesh filename="package://hbrs_gazebo_worlds/Media/models/brsu_home/livingroom_couch_2.dae" />
+				<mesh filename="package://hbrs_gazebo_worlds/common/objects/models/livingroom_couch_2.dae" />
 				<!-- <box size="2.83 0.95 0.68" /> -->
 			</geometry>
@@ -557,5 +557,5 @@
 			<origin xyz="0 0 0" />
 			<geometry>
-				<mesh filename="package://hbrs_gazebo_worlds/Media/models/brsu_home/livingroom_couch_3.dae" />
+				<mesh filename="package://hbrs_gazebo_worlds/common/objects/models/livingroom_couch_3.dae" />
 				<!-- <box size="0.93 1.55 0.66" /> -->
 			</geometry>
@@ -564,5 +564,5 @@
 			<origin xyz="0 0 0" />
 			<geometry>
-				<mesh filename="package://hbrs_gazebo_worlds/Media/models/brsu_home/livingroom_couch_3.dae" />
+				<mesh filename="package://hbrs_gazebo_worlds/common/objects/models/livingroom_couch_3.dae" />
 				<!-- <box size="0.95 1.57 0.68" /> -->
 			</geometry>
@@ -586,5 +586,5 @@
 			<origin xyz="0 0 0" />
 			<geometry>
-				<mesh filename="package://hbrs_gazebo_worlds/Media/models/brsu_home/livingroom_coffeetable.dae" />
+				<mesh filename="package://hbrs_gazebo_worlds/common/objects/models/livingroom_coffeetable.dae" />
 				<!-- <box size="1.205 0.582 0.40" /> -->
 			</geometry>
@@ -593,5 +593,5 @@
 			<origin xyz="0 0 0" />
 			<geometry>
-				<mesh filename="package://hbrs_gazebo_worlds/Media/models/brsu_home/livingroom_coffeetable.dae" />
+				<mesh filename="package://hbrs_gazebo_worlds/common/objects/models/livingroom_coffeetable.dae" />
 				<!-- <box size="1.225 0.602 0.42" /> -->
 			</geometry>
@@ -615,5 +615,5 @@
 			<origin xyz="0 0 0" />
 			<geometry>
-				<mesh filename="package://hbrs_gazebo_worlds/Media/models/brsu_home/desk.dae" />
+				<mesh filename="package://hbrs_gazebo_worlds/common/objects/models/desk.dae" />
 				<!-- <box size="1.60 0.80 0.72" /> -->
 			</geometry>
@@ -622,5 +622,5 @@
 			<origin xyz="0 0 0" />
 			<geometry>
-				<mesh filename="package://hbrs_gazebo_worlds/Media/models/brsu_home/desk.dae" />
+				<mesh filename="package://hbrs_gazebo_worlds/common/objects/models/desk.dae" />
 				<!-- <box size="1.62 0.82 0.74" /> -->
 			</geometry>
@@ -644,5 +644,5 @@
 			<origin xyz="0 0 0" />
 			<geometry>
-				<mesh filename="package://hbrs_gazebo_worlds/Media/models/brsu_home/charger_desk.dae" />
+				<mesh filename="package://hbrs_gazebo_worlds/common/objects/models/charger_desk.dae" />
 				<!-- <box size="0.45 0.45 0.50" /> -->
 			</geometry>
@@ -651,5 +651,5 @@
 			<origin xyz="0 0 0" />
 			<geometry>
-				<mesh filename="package://hbrs_gazebo_worlds/Media/models/brsu_home/charger_desk.dae" />
+				<mesh filename="package://hbrs_gazebo_worlds/common/objects/models/charger_desk.dae" />
 				<!-- <box size="0.47 0.47 0.52" /> -->
 			</geometry>
@@ -674,11 +674,11 @@
 			<origin xyz="0 0 0" />
 			<geometry>
-				<mesh filename="package://hbrs_gazebo_worlds/Media/models/brsu_home/diningroom_table.dae" />
-			</geometry>
-		</visual>
-		<collision>
-			<origin xyz="0 0 0" />
-			<geometry>
-				<mesh filename="package://hbrs_gazebo_worlds/Media/models/brsu_home/diningroom_table.dae" />
+				<mesh filename="package://hbrs_gazebo_worlds/common/objects/models/diningroom_table.dae" />
+			</geometry>
+		</visual>
+		<collision>
+			<origin xyz="0 0 0" />
+			<geometry>
+				<mesh filename="package://hbrs_gazebo_worlds/common/objects/models/diningroom_table.dae" />
 				<!-- <box size="2.21 1.02 0.76" /> -->
 			</geometry>
@@ -702,11 +702,11 @@
 			<origin xyz="0 0 0" />
 			<geometry>
-				<mesh filename="package://hbrs_gazebo_worlds/Media/models/brsu_home/diningroom_chair.dae" />
-			</geometry>
-		</visual>
-		<collision>
-			<origin xyz="0 0 0" />
-			<geometry>
-				<mesh filename="package://hbrs_gazebo_worlds/Media/models/brsu_home/diningroom_chair.dae" />
+				<mesh filename="package://hbrs_gazebo_worlds/common/objects/models/diningroom_chair.dae" />
+			</geometry>
+		</visual>
+		<collision>
+			<origin xyz="0 0 0" />
+			<geometry>
+				<mesh filename="package://hbrs_gazebo_worlds/common/objects/models/diningroom_chair.dae" />
 				<!-- <box size="0.547 0.52 0.99" /> -->
 			</geometry>
@@ -730,11 +730,11 @@
 			<origin xyz="0 0 0" />
 			<geometry>
-				<mesh filename="package://hbrs_gazebo_worlds/Media/models/brsu_home/diningroom_chair.dae" />
-			</geometry>
-		</visual>
-		<collision>
-			<origin xyz="0 0 0" />
-			<geometry>
-				<mesh filename="package://hbrs_gazebo_worlds/Media/models/brsu_home/diningroom_chair.dae" />
+				<mesh filename="package://hbrs_gazebo_worlds/common/objects/models/diningroom_chair.dae" />
+			</geometry>
+		</visual>
+		<collision>
+			<origin xyz="0 0 0" />
+			<geometry>
+				<mesh filename="package://hbrs_gazebo_worlds/common/objects/models/diningroom_chair.dae" />
 				<!-- <box size="0.547 0.52 0.99" /> -->
 			</geometry>
@@ -758,11 +758,11 @@
 			<origin xyz="0 0 0" />
 			<geometry>
-				<mesh filename="package://hbrs_gazebo_worlds/Media/models/brsu_home/diningroom_chair.dae" />
-			</geometry>
-		</visual>
-		<collision>
-			<origin xyz="0 0 0" />
-			<geometry>
-				<mesh filename="package://hbrs_gazebo_worlds/Media/models/brsu_home/diningroom_chair.dae" />
+				<mesh filename="package://hbrs_gazebo_worlds/common/objects/models/diningroom_chair.dae" />
+			</geometry>
+		</visual>
+		<collision>
+			<origin xyz="0 0 0" />
+			<geometry>
+				<mesh filename="package://hbrs_gazebo_worlds/common/objects/models/diningroom_chair.dae" />
 				<!-- <box size="0.547 0.52 0.99" /> -->
 			</geometry>
@@ -786,11 +786,11 @@
 			<origin xyz="0 0 0" />
 			<geometry>
-				<mesh filename="package://hbrs_gazebo_worlds/Media/models/brsu_home/diningroom_chair.dae" />
-			</geometry>
-		</visual>
-		<collision>
-			<origin xyz="0 0 0" />
-			<geometry>
-				<mesh filename="package://hbrs_gazebo_worlds/Media/models/brsu_home/diningroom_chair.dae" />
+				<mesh filename="package://hbrs_gazebo_worlds/common/objects/models/diningroom_chair.dae" />
+			</geometry>
+		</visual>
+		<collision>
+			<origin xyz="0 0 0" />
+			<geometry>
+				<mesh filename="package://hbrs_gazebo_worlds/common/objects/models/diningroom_chair.dae" />
 				<!-- <box size="0.547 0.52 0.99" /> -->
 			</geometry>
@@ -814,11 +814,11 @@
 			<origin xyz="0 0 0" />
 			<geometry>
-				<mesh filename="package://hbrs_gazebo_worlds/Media/models/brsu_home/diningroom_chair.dae" />
-			</geometry>
-		</visual>
-		<collision>
-			<origin xyz="0 0 0" />
-			<geometry>
-				<mesh filename="package://hbrs_gazebo_worlds/Media/models/brsu_home/diningroom_chair.dae" />
+				<mesh filename="package://hbrs_gazebo_worlds/common/objects/models/diningroom_chair.dae" />
+			</geometry>
+		</visual>
+		<collision>
+			<origin xyz="0 0 0" />
+			<geometry>
+				<mesh filename="package://hbrs_gazebo_worlds/common/objects/models/diningroom_chair.dae" />
 				<!-- <box size="0.547 0.52 0.99" /> -->
 			</geometry>
@@ -843,5 +843,5 @@
 			<origin xyz="0 0 0" />
 			<geometry>
-				<mesh filename="package://hbrs_gazebo_worlds/Media/models/brsu_home/middle_shelf.dae" />
+				<mesh filename="package://hbrs_gazebo_worlds/common/objects/models/middle_shelf.dae" />
 				<!-- <box size="0.44 2.42 0.80" /> -->
 			</geometry>
@@ -850,5 +850,5 @@
 			<origin xyz="0 0 0" />
 			<geometry>
-				<mesh filename="package://hbrs_gazebo_worlds/Media/models/brsu_home/middle_shelf.dae" />
+				<mesh filename="package://hbrs_gazebo_worlds/common/objects/models/middle_shelf.dae" />
 				<!-- <box size="0.46 2.44 0.82" /> -->
 			</geometry>
@@ -872,5 +872,5 @@
 			<origin xyz="0 0 0" />
 			<geometry>
-				<mesh filename="package://hbrs_gazebo_worlds/Media/models/brsu_home/middle_shelf.dae" />
+				<mesh filename="package://hbrs_gazebo_worlds/common/objects/models/middle_shelf.dae" />
 				<!-- <box size="0.44 2.42 0.80" /> -->
 			</geometry>
@@ -879,5 +879,5 @@
 			<origin xyz="0 0 0" />
 			<geometry>
-				<mesh filename="package://hbrs_gazebo_worlds/Media/models/brsu_home/middle_shelf.dae" />
+				<mesh filename="package://hbrs_gazebo_worlds/common/objects/models/middle_shelf.dae" />
 				<!-- <box size="0.46 2.44 0.82" /> -->
 			</geometry>
@@ -901,5 +901,5 @@
 			<origin xyz="0 0 0" />
 			<geometry>
-				<mesh filename="package://hbrs_gazebo_worlds/Media/models/brsu_home/middle_shelf.dae" />
+				<mesh filename="package://hbrs_gazebo_worlds/common/objects/models/middle_shelf.dae" />
 				<!-- <box size="0.44 2.42 0.80" /> -->
 			</geometry>
@@ -908,5 +908,5 @@
 			<origin xyz="0 0 0" />
 			<geometry>
-				<mesh filename="package://hbrs_gazebo_worlds/Media/models/brsu_home/middle_shelf.dae" />
+				<mesh filename="package://hbrs_gazebo_worlds/common/objects/models/middle_shelf.dae" />
 				<!-- <box size="0.46 2.44 0.82" /> -->
 			</geometry>
@@ -930,5 +930,5 @@
 			<origin xyz="0 0 0" />
 			<geometry>
-				<mesh filename="package://hbrs_gazebo_worlds/Media/models/brsu_home/middle_shelf.dae" />
+				<mesh filename="package://hbrs_gazebo_worlds/common/objects/models/middle_shelf.dae" />
 				<!-- <box size="0.44 2.42 0.80" /> -->
 			</geometry>
@@ -937,5 +937,5 @@
 			<origin xyz="0 0 0" />
 			<geometry>
-				<mesh filename="package://hbrs_gazebo_worlds/Media/models/brsu_home/middle_shelf.dae" />
+				<mesh filename="package://hbrs_gazebo_worlds/common/objects/models/middle_shelf.dae" />
 				<!-- <box size="0.46 2.44 0.82" /> -->
 			</geometry>
@@ -959,5 +959,5 @@
 			<origin xyz="0 0 0" />
 			<geometry>
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
Commit message: small fixes for simulation

File: hbrs_environments/hbrs_gazebo_worlds/common/worlds/brsu-c069.urdf.xacro (robot description, xacro)
@@ -49,7 +49,4 @@
 		</collision>
 	</link>
-	<gazebo reference="north_wall">
-		<material>BRSU/Wall</material>
-	</gazebo>
 	<joint name="joint_north_wall" type="fixed">
 		<origin xyz="-0.25 4.06 1.30" rpy="0 0 0" />
@@ -77,7 +74,4 @@
 		</collision>
 	</link>
-	<gazebo reference="east_wall">
-		<material>BRSU/Wall</material>
-	</gazebo>
 	<joint name="joint_east_wall" type="fixed">
 		<origin xyz="7.40 0.59 1.30" rpy="0 0 0" />
@@ -105,7 +99,4 @@
 		</collision>
 	</link>
-	<gazebo reference="south_wall">
-		<material>BRSU/Wall</material>
-	</gazebo>
 	<joint name="joint_south_wall" type="fixed">
 		<origin xyz="-0.25 -2.88 1.30" rpy="0 0 0" />
@@ -133,7 +124,4 @@
 		</collision>
 	</link>
-	<gazebo reference="west_wall">
-		<material>BRSU/Wall</material>
-	</gazebo>
 	<joint name="joint_west_wall" type="fixed">
 		<origin xyz="-7.90 0.59 1.30" rpy="0 0 0" />
@@ -161,7 +149,4 @@
 		</collision>
 	</link>
-	<gazebo reference="west_divider">
-		<material>BRSU/Wall</material>
-	</gazebo>
 	<joint name="joint_west_divider" type="fixed">
 		<origin xyz="-5.84 0.218 1.30" rpy="0 0 0" />
@@ -979,4 +964,4 @@
 	</joint>
 </xacro:macro>
-<xacro:brsu_home name="brsu_home" />
+<xacro:brsu-c069 name="brsu-c069" />
 </robot>
