Commit message: adjust folder structure of gazebo objects package according to our guidelines

File: hbrs_environments/hbrs_gazebo_objects/ros/templates/model.urdf.xacro (robot description, xacro)
@@ -24,5 +24,5 @@
 				<origin xyz="0 0 ${-size_z/2}" rpy="0 0 0" />
 				<geometry>
-					<mesh filename="package://hbrs_gazebo_objects/models/${model_filename}" scale="${scale} ${scale} ${scale}" />
+					<mesh filename="package://hbrs_gazebo_objects/common/models/${model_filename}" scale="${scale} ${scale} ${scale}" />
 				</geometry>
 			</visual>

File: hbrs_environments/hbrs_gazebo_objects/ros/templates/screw.urdf.xacro (robot description, xacro)
@@ -1,6 +1,6 @@
 <?xml version="1.0"?>
 <robot name="screw_template" xmlns:xacro="http://ros.org/wiki/xacro">
-	<include filename="$(find hbrs_gazebo_objects)/templates/pipe.urdf.xacro" />
-	<include filename="$(find hbrs_gazebo_objects)/templates/nut.urdf.xacro" />
+	<include filename="$(find hbrs_gazebo_objects)/ros/templates/pipe.urdf.xacro" />
+	<include filename="$(find hbrs_gazebo_objects)/ros/templates/nut.urdf.xacro" />
 	<xacro:macro name="screw_template" params="name length radius color">
 		<xacro:pipe_template name="pipe_20" radius="${radius / 2}" height="${length}" color="Gazebo/Black" />

File: hbrs_environments/hbrs_gazebo_objects/ros/urdf/adapter_sleeve_r20.urdf.xacro (robot description, xacro)
@@ -1,5 +1,5 @@
 <?xml version="1.0"?>
 <robot name="adapter_sleeve_r20" xmlns:xacro="http://ros.org/wiki/xacro">
-	<include filename="$(find hbrs_gazebo_objects)/templates/model.urdf.xacro" />
+	<include filename="$(find hbrs_gazebo_objects)/ros/templates/model.urdf.xacro" />
 	<xacro:model_template name="adapter_sleeve_r20" model_filename="adapter_sleeve_r20.dae" scale="0.001" size_x="0.03" size_y="0.03" size_z="0.045" weight="0.010"/>
 </robot>

File: hbrs_environments/hbrs_gazebo_objects/ros/urdf/adapter_sleeve_v20.urdf.xacro (robot description, xacro)
@@ -1,5 +1,5 @@
 <?xml version="1.0"?>
 <robot name="adapter_sleeve_v20" xmlns:xacro="http://ros.org/wiki/xacro">
-	<include filename="$(find hbrs_gazebo_objects)/templates/model.urdf.xacro" />
+	<include filename="$(find hbrs_gazebo_objects)/ros/templates/model.urdf.xacro" />
 	<xacro:model_template name="adapter_sleeve_v20" model_filename="adapter_sleeve_v20.dae" scale="0.001" size_x="0.03" size_y="0.03" size_z="0.045" weight="0.015"/>
 </robot>

File: hbrs_environments/hbrs_gazebo_objects/ros/urdf/aluprofil_f20_100_gray.urdf.xacro (robot description, xacro)
@@ -1,5 +1,5 @@
 <?xml version="1.0"?>
 <robot name="aluprofil_f20_100_gray" xmlns:xacro="http://ros.org/wiki/xacro">
-	<include filename="$(find hbrs_gazebo_objects)/templates/model.urdf.xacro" />
+	<include filename="$(find hbrs_gazebo_objects)/ros/templates/model.urdf.xacro" />
 	<xacro:model_template name="aluprofil_f20_100_gray" model_filename="aluprofil_f20_100_gray.dae" scale="0.001"  size_x="0.02" size_y="0.02" size_z="0.1" weight="0.05"/>
 </robot>

File: hbrs_environments/hbrs_gazebo_objects/ros/urdf/aluprofil_s40_100_gray.urdf.xacro (robot description, xacro)
@@ -1,5 +1,5 @@
 <?xml version="1.0"?>
 <robot name="aluprofil_s40_100_gray" xmlns:xacro="http://ros.org/wiki/xacro">
-	<include filename="$(find hbrs_gazebo_objects)/templates/model.urdf.xacro" />
+	<include filename="$(find hbrs_gazebo_objects)/ros/templates/model.urdf.xacro" />
 	<xacro:model_template name="aluprofil_s40_100_gray" model_filename="aluprofil_s40_100_gray.dae" scale="0.001"  size_x="0.04" size_y="0.04" size_z="0.1" weight="0.185"/>
 </robot>

File: hbrs_environments/hbrs_gazebo_objects/ros/urdf/bolt_m20_100.urdf.xacro (robot description, xacro)
@@ -1,5 +1,5 @@
 <?xml version="1.0"?>
 <robot name="bolt_m20_100" xmlns:xacro="http://ros.org/wiki/xacro">
-	<include filename="$(find hbrs_gazebo_objects)/templates/model.urdf.xacro" />
+	<include filename="$(find hbrs_gazebo_objects)/ros/templates/model.urdf.xacro" />
 	<xacro:model_template name="bolt_m20_100" model_filename="bolt_m20_100.dae" scale="0.001"  size_x="0.11" size_y="0.02" size_z="0.02" weight="0.290"/>
 </robot>

File: hbrs_environments/hbrs_gazebo_objects/ros/urdf/bolt_m20_180.urdf.xacro (robot description, xacro)
@@ -1,5 +1,5 @@
 <?xml version="1.0"?>
 <robot name="bolt_m20_180" xmlns:xacro="http://ros.org/wiki/xacro">
-	<include filename="$(find hbrs_gazebo_objects)/templates/model.urdf.xacro" />
+	<include filename="$(find hbrs_gazebo_objects)/ros/templates/model.urdf.xacro" />
 	<xacro:model_template name="bolt_m20_180" model_filename="bolt_m20_180.dae" scale="0.001"  size_x="0.11" size_y="0.02" size_z="0.02" weight="0.477"/>
 </robot>

File: hbrs_environments/hbrs_gazebo_objects/ros/urdf/nut_m20.urdf.xacro (robot description, xacro)
@@ -1,5 +1,5 @@
 <?xml version="1.0"?>
 <robot name="nut_m20" xmlns:xacro="http://ros.org/wiki/xacro">
-	<include filename="$(find hbrs_gazebo_objects)/templates/model.urdf.xacro" />
+	<include filename="$(find hbrs_gazebo_objects)/ros/templates/model.urdf.xacro" />
 	<xacro:model_template name="nut_m20" model_filename="nut_m20.dae" scale="0.001"  size_x="0.015" size_y="0.028" size_z="0.028" weight="0.068"/>
 </robot>

File: hbrs_environments/hbrs_gazebo_objects/ros/urdf/nut_m30.urdf.xacro (robot description, xacro)
@@ -1,5 +1,5 @@
 <?xml version="1.0"?>
 <robot name="nut_m30" xmlns:xacro="http://ros.org/wiki/xacro">
-	<include filename="$(find hbrs_gazebo_objects)/templates/model.urdf.xacro" />
+	<include filename="$(find hbrs_gazebo_objects)/ros/templates/model.urdf.xacro" />
 	<xacro:model_template name="nut_m30" model_filename="nut_m30.dae" scale="0.001"  size_x="0.025" size_y="0.045" size_z="0.045"  weight="0.215"/>
 </robot>
